File: Kicad/esp-nes.kicad_pcb (KiCad board)
At the start: 2 copper layers, 189.5 x 67 mm, 11 parts, among them U1 ESP32-DevKitC, U2 CR2013-MI2120, U3 pam8403

Commit message: updata file
Parts:
- renumbered A to A1, B to B1, DOWN to DOWN1, LEFT to LEFT1, RIGHT to RIGHT1, SELECT to SELECT1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
Connections:
- U3 pad 2: unconnected-(U3-T-Pad2) -> GND
- U3 pad 3: unconnected-(U3-R-Pad3) -> L
Routing:
- net L: track 40.6 -> 46.5 mm
